File: schematic/drone-power-supply-v2.kicad_pcb (KiCad board)
At the start: 2 copper layers, 52 parts, among them J1 5V, J2 6V, J3 12V, J4 Battery, U1 TPS54360DDA, U2 TPS54360DDA, U3 TPS54360DDA

Commit message: push latest changes
Parts:
- added J5: POWER_PAD, drone-power-supply-v2:PCB_WirePad_5mm, F.Cu at (162.2, 110.0)
- added MT1: MOUNT_HOLE, MountingHole:MountingHole_3.2mm_M3_Pad, F.Cu at (161.5, 117.5)
- added MT2: MOUNT_HOLE, MountingHole:MountingHole_3.2mm_M3_Pad, F.Cu at (161.5, 80.5)
- added MT3: MOUNT_HOLE, MountingHole:MountingHole_3.2mm_M3_Pad, F.Cu at (124.5, 80.5)
- added MT4: MOUNT_HOLE, MountingHole:MountingHole_3.2mm_M3_Pad, F.Cu at (124.5, 117.5)
- C10, C11, C17, C18, C3, C4: value 10uF 63V -> CAP_10uF_63V; footprint Capacitors_SMD:C_1210 -> CAPC:CAPC3225X25N
- C12: value 18pF 10V -> CAP_39pF_16V; footprint Capacitors_SMD:C_0603 -> CAPC:CAPC1608X09N
- C13, C14, C20, C21, C6, C7: value 47uF 16V -> CAP_47uF_16V; footprint Capacitors_SMD:C_1210 -> CAPC:CAPC3225X25N
- C15, C8: value 6800pF 10V -> CAP_8200pF_10V; footprint Capacitors_SMD:C_0603 -> CAPC:CAPC1608X09N
- C16, C2, C9: value 0.1uF 16V -> CAP_100nF_10V; footprint Capacitors_SMD:C_0603 -> CAPC:CAPC1608X09N
- C19: value 13pF 10V -> CAP_39pF_16V; footprint Capacitors_SMD:C_0603 -> CAPC:CAPC1608X09N
- C22: value 8200pF 50V -> CAP_8200pF_10V; footprint Capacitors_SMD:C_0603 -> CAPC:CAPC1608X09N
- C5: value 39pF 16V -> CAP_39pF_16V; footprint Capacitors_SMD:C_0603 -> CAPC:CAPC1608X09N
- D1, D2, D3: value B560C 60V 5A -> D_B520C; footprint Diodes_SMD:D_SMC -> DIOM:DIOM7162X25N
- J1: value 5V -> POWER_PAD; footprint Wire_Pads:SolderWirePad_single_SMD_5x10mm -> drone-power-supply-v2:PCB_WirePad_5mm
- J2: value 6V -> POWER_PAD; footprint Wire_Pads:SolderWirePad_single_SMD_5x10mm -> drone-power-supply-v2:PCB_WirePad_5mm
- J3: value 12V -> POWER_PAD; footprint Wire_Pads:SolderWirePad_single_SMD_5x10mm -> drone-power-supply-v2:PCB_WirePad_5mm
- J4: value Battery -> CONN_XT60; footprint Connectors:XT60 -> drone-power-supply-v2:XT60
- L1, L2: value 8.2uH 4.5A -> L_8.2uH_4.5A; footprint Inductors_SMD:6540 -> INDM:INDM7265X40N
- L3: value 15uH 4.6A -> L_15uH_5A; footprint Inductors_SMD:L_1260 -> INDM:INDM125125X60N
- R1, R13, R7: value 523k 1% -> RES_523K_1%; footprint Resistors_SMD:R_0603 -> RESC:RESC1608X04N
- R10, R16: value 100k 1% -> RES_100K_1%; footprint Resistors_SMD:R_0603 -> RESC:RESC1608X04N
- R11, R17, R5: value 84.5k 1% -> RES_84.5K_1%; footprint Resistors_SMD:R_0603 -> RESC:RESC1608X04N
- R12, R18, R6: value 10k2 1% -> RES_10.2K_1%; footprint Resistors_SMD:R_0603 -> RESC:RESC1608X04N
- R14: value 143k 1% -> RES_143K_1%; footprint Resistors_SMD:R_0603 -> RESC:RESC1608X04N
- R15: value 25k5 1% -> RES_25.5K_1%; footprint Resistors_SMD:R_0603 -> RESC:RESC1608X04N
- R2: value 53.6k 1% -> RES_53.6K_1%; footprint Resistors_SMD:R_0603 -> RESC:RESC1608X04N
- R3: value 13k 1% -> RES_13K_1%; footprint Resistors_SMD:R_0603 -> RESC:RESC1608X04N
- R4: value 162k 1% -> RES_162K_1%; footprint Resistors_SMD:R_0603 -> RESC:RESC1608X04N
- R8: value 66k5 1% -> RES_66.5K_1%; footprint Resistors_SMD:R_0603 -> RESC:RESC1608X04N
- R9: value 18k 1% -> RES_18K_1%; footprint Resistors_SMD:R_0603 -> RESC:RESC1608X04N
- U1, U2, U3: footprint Housings_SOIC:TI_SO-PowerPAD-8 -> SOIC:SOIC127P600X175_HS-9N
- moved J1 77.7 mm to (162.2, 89.0)
- moved L2 75.6 mm to (152.8, 96.5)
- moved J2 72.8 mm to (162.2, 96.0)
- moved C20 72.7 mm to (156.0, 110.7), turned to 0 degrees
- moved R8 72.1 mm to (150.8, 106.5), turned to 0 degrees
- moved D2 72.0 mm to (142.5, 96.5)
- moved L3 71.6 mm to (144.7, 114.2), turned to 0 degrees
- moved C4 71.6 mm to (134.6, 87.6), turned to 90 degrees
- moved J4 71.5 mm to (124.9, 97.7)
- moved R2 71.5 mm to (148.2, 92.0), turned to 0 degrees
- moved C21 70.3 mm to (156.0, 114.0), turned to 0 degrees
- moved R10 70.2 mm to (142.5, 106.5), turned to 0 degrees
- moved R7 69.9 mm to (139.0, 103.2)
- moved C14 69.8 mm to (155.8, 103.1)
- moved C13 69.7 mm to (152.4, 103.1)
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Connections:
- net Net-(C13-Pad1) renamed /PWR_OUT_6V
- net Net-(C16-Pad2) renamed /PWR_12V_SW
- net Net-(C2-Pad2) renamed /PWR_5V_SW
- net Net-(C20-Pad1) renamed /PWR_OUT_12V
- net Net-(C6-Pad1) renamed /PWR_OUT_5V
- net Net-(C9-Pad2) renamed /PWR_6V_SW
Routing:
- net VBAT: track 0.00 -> 56.1 mm
- net /PWR_OUT_12V: track 0.00 -> 40.1 mm
- net /PWR_OUT_5V: track 0.00 -> 26.2 mm
- net /PWR_OUT_6V: track 0.00 -> 26.0 mm
- net /PWR_12V_SW: track 0.00 -> 20.4 mm
- net /PWR_6V_SW: track 0.00 -> 16.8 mm
- net Net-(R14-Pad2): track 0.00 -> 15.6 mm
- net /PWR_5V_SW: track 0.00 -> 14.5 mm
- net Net-(R2-Pad2): track 0.00 -> 9.08 mm
- net Net-(R12-Pad1): track 0.00 -> 8.31 mm
- net Net-(C19-Pad1): track 0.00 -> 6.86 mm
- net Net-(C5-Pad1): track 0.00 -> 3.48 mm
- net Net-(C12-Pad1): track 0.00 -> 3.48 mm
- net GND: track 0.00 -> 3.35 mm, vias 0 -> 176
- net Net-(R1-Pad2): track 0.00 -> 3.30 mm
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- added copper zone on B.Cu, net GND
- added copper zone on F.Cu, net GND
Other:
- board outline added: 45 x 45 mm
- net class Default: trace_width 0.25 -> 0.3
- net class HIGH_POWER added: clearance 0.2, trace_width 7.82937, via_dia 0.9, via_drill 0.5
- net class POWER added: clearance 0.2, trace_width 1.72, via_dia 0.8, via_drill 0.4
- rule trace_min: 0.2 -> 0.1524
- board text added: "12V"
- board text added: "5V"
- board text added: "6V"
- board text added: "GND"
