File: schematic/drone-power-supply-v2.sch (KiCad schematic (older format))
At the start: 17 parts

Commit message: add initial board placement and 6 + 12v regulators
Parts:
- removed C?: 100uF 63V, symbol device:CP_Small
- added C10, C11, C17, C18, C4: 10uF 63V, Capacitors_SMD:C_1210, symbol drone-power-supply-v2-rescue:C_Small-device
- added C12: 18pF 10V, Capacitors_SMD:C_0603, symbol drone-power-supply-v2-rescue:C_Small-device
- added C13, C14, C20, C21: 47uF 16V, Capacitors_SMD:C_1210, symbol drone-power-supply-v2-rescue:C_Small-device
- added C15: 6800pF 10V, Capacitors_SMD:C_0603, symbol drone-power-supply-v2-rescue:C_Small-device
- added C16, C9: 0.1uF 16V, Capacitors_SMD:C_0603, symbol drone-power-supply-v2-rescue:C_Small-device
- added C19: 13pF 10V, Capacitors_SMD:C_0603, symbol drone-power-supply-v2-rescue:C_Small-device
- added C22: 8200pF 50V, Capacitors_SMD:C_0603, symbol drone-power-supply-v2-rescue:C_Small-device
- added D2, D3: B560C 60V 5A, Diodes_SMD:D_SMC, symbol drone-power-supply-v2-rescue:D_Small_ALT-device
- added J2: 6V, Wire_Pads:SolderWirePad_single_SMD_5x10mm, symbol drone-power-supply-v2-rescue:Conn_01x01-Connector
- added J3: 12V, Wire_Pads:SolderWirePad_single_SMD_5x10mm, symbol drone-power-supply-v2-rescue:Conn_01x01-Connector
- added J4: Battery, Connectors:XT60, symbol Connector:Conn_01x02
- added L2: 8.2uH 4.5A, Inductors_SMD:6540, symbol drone-power-supply-v2-rescue:L_Small-device
- added L3: 15uH 4.6A, Inductors_SMD:L_1260, symbol drone-power-supply-v2-rescue:L_Small-device
- added R10, R16: 100k 1%, Resistors_SMD:R_0603, symbol drone-power-supply-v2-rescue:R_Small-device
- added R11, R17: 84.5k 1%, Resistors_SMD:R_0603, symbol drone-power-supply-v2-rescue:R_Small-device
- added R12, R18: 10k2 1%, Resistors_SMD:R_0603, symbol drone-power-supply-v2-rescue:R_Small-device
- added R13, R7: 523k 1%, Resistors_SMD:R_0603, symbol drone-power-supply-v2-rescue:R_Small-device
- added R14: 143k 1%, Resistors_SMD:R_0603, symbol drone-power-supply-v2-rescue:R_Small-device
- added R15: 25k5 1%, Resistors_SMD:R_0603, symbol drone-power-supply-v2-rescue:R_Small-device
- added R8: 66k5 1%, Resistors_SMD:R_0603, symbol drone-power-supply-v2-rescue:R_Small-device
- added R9: 18k 1%, Resistors_SMD:R_0603, symbol drone-power-supply-v2-rescue:R_Small-device
- added U2, U3: TPS54360DDA, Housings_SOIC:TI_SO-PowerPAD-8, symbol drone-power-supply-v2-rescue:TPS54360DDA-dc-dc
- C2: renamed from C?; value 2.2uF 63V -> 0.1uF 16V; footprint (none) -> Capacitors_SMD:C_0603; symbol device:C_Small -> drone-power-supply-v2-rescue:C_Small-device
- C3: renamed from C?; value 2.2uF 63V -> 10uF 63V; footprint (none) -> Capacitors_SMD:C_1210; symbol device:C_Small -> drone-power-supply-v2-rescue:C_Small-device
- C5: renamed from C?; value 39pF -> 39pF 16V; footprint (none) -> Capacitors_SMD:C_0603; symbol device:C_Small -> drone-power-supply-v2-rescue:C_Small-device
- C6, C7: renamed from C?; value 47uF 10V -> 47uF 16V; footprint (none) -> Capacitors_SMD:C_1210; symbol device:C_Small -> drone-power-supply-v2-rescue:C_Small-device
- C8: renamed from C?; value 6800pF -> 6800pF 10V; footprint (none) -> Capacitors_SMD:C_0603; symbol device:C_Small -> drone-power-supply-v2-rescue:C_Small-device
- D1: renamed from D?; footprint (none) -> Diodes_SMD:D_SMC; symbol device:D_Small_ALT -> drone-power-supply-v2-rescue:D_Small_ALT-device
- J1: renamed from J?; footprint (none) -> Wire_Pads:SolderWirePad_single_SMD_5x10mm; symbol Connector:Conn_01x01 -> drone-power-supply-v2-rescue:Conn_01x01-Connector
- L1: renamed from L?; footprint (none) -> Inductors_SMD:6540; symbol device:L_Small -> drone-power-supply-v2-rescue:L_Small-device
- R1: renamed from R?; value 523k -> 523k 1%; footprint (none) -> Resistors_SMD:R_0603; symbol device:R_Small -> drone-power-supply-v2-rescue:R_Small-device
- R2: renamed from R?; value 523k -> 53.6k 1%; footprint (none) -> Resistors_SMD:R_0603; symbol device:R_Small -> drone-power-supply-v2-rescue:R_Small-device
- R3: renamed from R?; value 13k -> 13k 1%; footprint (none) -> Resistors_SMD:R_0603; symbol device:R_Small -> drone-power-supply-v2-rescue:R_Small-device
- R4: renamed from R?; value 162k -> 162k 1%; footprint (none) -> Resistors_SMD:R_0603; symbol device:R_Small -> drone-power-supply-v2-rescue:R_Small-device
- R5: renamed from R?; value 84.5k -> 84.5k 1%; footprint (none) -> Resistors_SMD:R_0603; symbol device:R_Small -> drone-power-supply-v2-rescue:R_Small-device
- R6: renamed from R?; footprint (none) -> Resistors_SMD:R_0603; symbol device:R_Small -> drone-power-supply-v2-rescue:R_Small-device
- U1: renamed from U?; footprint Housings_SOIC:TI_SO-PowerPAD-8_ThermalVias -> Housings_SOIC:TI_SO-PowerPAD-8; symbol dc-dc:TPS54360DDA -> drone-power-supply-v2-rescue:TPS54360DDA-dc-dc
Connections:
- wire segments 56 -> 171
Other:
- note added: "50V cap more common than 10V so use it if 10V is not available."
- note added: "F = 600kHz"
- note added: "F = 960kHz"
- note added: "Rt"

Commit message: push latest changes
Parts:
- added J5: POWER_PAD, drone-power-supply-v2:PCB_WirePad_5mm, symbol drone-power-supply-v2:POWER_PAD
- added MT1, MT2, MT3, MT4: MOUNT_HOLE, MountingHole:MountingHole_3.2mm_M3_Pad, symbol drone-power-supply-v2:MOUNT_HOLE
- C10, C11, C17, C18, C3, C4: value 10uF 63V -> CAP_10uF_63V; footprint Capacitors_SMD:C_1210 -> CAPC:CAPC3225X25N; symbol drone-power-supply-v2-rescue:C_Small-device -> drone-power-supply-v2:CAP_10uF_63V; MFN (none) -> GRM32ER71J106KA12L
- C12: value 18pF 10V -> CAP_39pF_16V; footprint Capacitors_SMD:C_0603 -> CAPC:CAPC1608X09N; symbol drone-power-supply-v2-rescue:C_Small-device -> drone-power-supply-v2:CAP_39pF_16V; MFN (none) -> C0603C390J5GACTU
- C13, C14, C20, C21, C6, C7: value 47uF 16V -> CAP_47uF_16V; footprint Capacitors_SMD:C_1210 -> CAPC:CAPC3225X25N; symbol drone-power-supply-v2-rescue:C_Small-device -> drone-power-supply-v2:CAP_47uF_16V; MFN (none) -> EMK325BJ476MM-T
- C15, C8: value 6800pF 10V -> CAP_8200pF_10V; footprint Capacitors_SMD:C_0603 -> CAPC:CAPC1608X09N; symbol drone-power-supply-v2-rescue:C_Small-device -> drone-power-supply-v2:CAP_8200pF_10V; MFN (none) -> VJ0603Y822KXAPW1BC
- C16, C2, C9: value 0.1uF 16V -> CAP_100nF_10V; footprint Capacitors_SMD:C_0603 -> CAPC:CAPC1608X09N; symbol drone-power-supply-v2-rescue:C_Small-device -> drone-power-supply-v2:CAP_100nF_10V; MFN (none) -> VJ0603Y104JXQPW1BC
- C19: value 13pF 10V -> CAP_39pF_16V; footprint Capacitors_SMD:C_0603 -> CAPC:CAPC1608X09N; symbol drone-power-supply-v2-rescue:C_Small-device -> drone-power-supply-v2:CAP_39pF_16V; MFN (none) -> C0603C390J5GACTU
- C22: value 8200pF 50V -> CAP_8200pF_10V; footprint Capacitors_SMD:C_0603 -> CAPC:CAPC1608X09N; symbol drone-power-supply-v2-rescue:C_Small-device -> drone-power-supply-v2:CAP_8200pF_10V; MFN (none) -> VJ0603Y822KXAPW1BC
- C5: value 39pF 16V -> CAP_39pF_16V; footprint Capacitors_SMD:C_0603 -> CAPC:CAPC1608X09N; symbol drone-power-supply-v2-rescue:C_Small-device -> drone-power-supply-v2:CAP_39pF_16V; MFN (none) -> C0603C390J5GACTU
- D1, D2, D3: value B560C 60V 5A -> D_B520C; footprint Diodes_SMD:D_SMC -> DIOM:DIOM7162X25N; symbol drone-power-supply-v2-rescue:D_Small_ALT-device -> drone-power-supply-v2:D_B520C; MFN (none) -> B520C-13-F
- J1: value 5V -> POWER_PAD; footprint Wire_Pads:SolderWirePad_single_SMD_5x10mm -> drone-power-supply-v2:PCB_WirePad_5mm; symbol drone-power-supply-v2-rescue:Conn_01x01-Connector -> drone-power-supply-v2:POWER_PAD
- J2: value 6V -> POWER_PAD; footprint Wire_Pads:SolderWirePad_single_SMD_5x10mm -> drone-power-supply-v2:PCB_WirePad_5mm; symbol drone-power-supply-v2-rescue:Conn_01x01-Connector -> drone-power-supply-v2:POWER_PAD
- J3: value 12V -> POWER_PAD; footprint Wire_Pads:SolderWirePad_single_SMD_5x10mm -> drone-power-supply-v2:PCB_WirePad_5mm; symbol drone-power-supply-v2-rescue:Conn_01x01-Connector -> drone-power-supply-v2:POWER_PAD
- J4: value Battery -> CONN_XT60; footprint Connectors:XT60 -> drone-power-supply-v2:XT60; symbol Connector:Conn_01x02 -> drone-power-supply-v2:CONN_XT60; Silkscreen (none) -> BATTERY
- L1, L2: value 8.2uH 4.5A -> L_8.2uH_4.5A; footprint Inductors_SMD:6540 -> INDM:INDM7265X40N; symbol drone-power-supply-v2-rescue:L_Small-device -> drone-power-supply-v2:L_8.2uH_4.5A; MFN (none) -> SRP6540-8R2M
- L3: value 15uH 4.6A -> L_15uH_5A; footprint Inductors_SMD:L_1260 -> INDM:INDM125125X60N; symbol drone-power-supply-v2-rescue:L_Small-device -> drone-power-supply-v2:L_15uH_5A; MFN (none) -> SRR1260A-150M
- R1, R13, R7: value 523k 1% -> RES_523K_1%; footprint Resistors_SMD:R_0603 -> RESC:RESC1608X04N; symbol drone-power-supply-v2-rescue:R_Small-device -> drone-power-supply-v2:RES_523K_1%; Field5 (none) -> Test; MFN (none) -> AC0603FR-07523KL
- R10, R16: value 100k 1% -> RES_100K_1%; footprint Resistors_SMD:R_0603 -> RESC:RESC1608X04N; symbol drone-power-supply-v2-rescue:R_Small-device -> drone-power-supply-v2:RES_100K_1%; MFN (none) -> CPF0603F100KC1
- R11, R17, R5: value 84.5k 1% -> RES_84.5K_1%; footprint Resistors_SMD:R_0603 -> RESC:RESC1608X04N; symbol drone-power-supply-v2-rescue:R_Small-device -> drone-power-supply-v2:RES_84.5K_1%; MFN (none) -> CR0603-FX-8452ELF
- R12, R18, R6: value 10k2 1% -> RES_10.2K_1%; footprint Resistors_SMD:R_0603 -> RESC:RESC1608X04N; symbol drone-power-supply-v2-rescue:R_Small-device -> drone-power-supply-v2:RES_10.2K_1%; MFN (none) -> RC0201FR-0710K2L
- R14: value 143k 1% -> RES_143K_1%; footprint Resistors_SMD:R_0603 -> RESC:RESC1608X04N; symbol drone-power-supply-v2-rescue:R_Small-device -> drone-power-supply-v2:RES_143K_1%; MFN (none) -> CR0603-FX-1433ELF
- R15: value 25k5 1% -> RES_25.5K_1%; footprint Resistors_SMD:R_0603 -> RESC:RESC1608X04N; symbol drone-power-supply-v2-rescue:R_Small-device -> drone-power-supply-v2:RES_25.5K_1%; MFN (none) -> CPF0603F25K5C1
- R2: value 53.6k 1% -> RES_53.6K_1%; footprint Resistors_SMD:R_0603 -> RESC:RESC1608X04N; symbol drone-power-supply-v2-rescue:R_Small-device -> drone-power-supply-v2:RES_53.6K_1%; MFN (none) -> CRCW060353K6FKEA
- R3: value 13k 1% -> RES_13K_1%; footprint Resistors_SMD:R_0603 -> RESC:RESC1608X04N; symbol drone-power-supply-v2-rescue:R_Small-device -> drone-power-supply-v2:RES_13K_1%; MFN (none) -> AC0603FR-0713KL
- R4: value 162k 1% -> RES_162K_1%; footprint Resistors_SMD:R_0603 -> RESC:RESC1608X04N; symbol drone-power-supply-v2-rescue:R_Small-device -> drone-power-supply-v2:RES_162K_1%; MFN (none) -> CRCW0603162KFKEA
- R8: value 66k5 1% -> RES_66.5K_1%; footprint Resistors_SMD:R_0603 -> RESC:RESC1608X04N; symbol drone-power-supply-v2-rescue:R_Small-device -> drone-power-supply-v2:RES_66.5K_1%; MFN (none) -> CPF0603F66K5C1
- R9: value 18k 1% -> RES_18K_1%; footprint Resistors_SMD:R_0603 -> RESC:RESC1608X04N; symbol drone-power-supply-v2-rescue:R_Small-device -> drone-power-supply-v2:RES_18K_1%; MFN (none) -> RN731JTTD1802F100
- U1, U2, U3: footprint Housings_SOIC:TI_SO-PowerPAD-8 -> SOIC:SOIC127P600X175_HS-9N; symbol drone-power-supply-v2-rescue:TPS54360DDA-dc-dc -> drone-power-supply-v2:TPS54360DDA; MFN (none) -> TPS54360DDA
Connections:
- net labels added: GND-power, PWR_12V_SW, PWR_5V_SW, PWR_6V_SW, PWR_OUT_12V, PWR_OUT_5V, PWR_OUT_6V
- wire segments 171 -> 172
- no-connect marks 0 -> 4
Other:
- note removed: "50V cap more common than 10V so use it if 10V is not available."
